File: Switch Lock/Switch Lock.kicad_pcb (KiCad board)
At the start: 2 copper layers, 1 part, among them J1 Conn_01x06

Commit message: finisheddesign
Parts:
- removed J1: Conn_01x06, Connector_PinHeader_2.54mm:PinHeader_1x06_P2.54mm_Vertical
- added J2: Conn_01x07, Connector_PinHeader_2.54mm:PinHeader_1x07_P2.54mm_Vertical, F.Cu at (107.5, 68.7)
- added R1: 2.2k, Resistor_SMD:R_0805_2012Metric_Pad1.20x1.40mm_HandSolder, F.Cu at (98.2, 68.7)
- added REF**: MountingHole_2.2mm_M2, MountingHole:MountingHole_2.2mm_M2, F.Cu at (127.7, 60.8)
- added REF**: MountingHole_2.2mm_M2, MountingHole:MountingHole_2.2mm_M2, F.Cu at (96.5, 60.2)
- added S1: JS102011SAQN, JS102011SAQN:SW_JS102011SAQN, F.Cu at (96.9, 79.7)
- added S2: JS102011SAQN, JS102011SAQN:SW_JS102011SAQN, F.Cu at (107.1, 79.7)
- added S3: JS102011SAQN, JS102011SAQN:SW_JS102011SAQN, F.Cu at (117.2, 79.6)
- added S4: JS102011SAQN, JS102011SAQN:SW_JS102011SAQN, F.Cu at (127.2, 79.6)
- added Status1: JS102011SAQN, JS102011SAQN:SW_JS102011SAQN, F.Cu at (117.8, 57.9)
Routing:
- net Net-(J2-Pin_2): track 0.00 -> 20.1 mm
- net GND: track 0.00 -> 14.0 mm, vias 0 -> 5
- net Net-(J2-Pin_3): track 0.00 -> 13.2 mm
- net Net-(J2-Pin_5): track 0.00 -> 11.7 mm
- net Net-(J2-Pin_4): track 0.00 -> 8.34 mm
- net Net-(J2-Pin_1): track 0.00 -> 8.29 mm
- net Net-(J2-Pin_6): track 0.00 -> 8.06 mm
- added copper zone on F.Cu, net /3.3v
- added copper zone on B.Cu, net GND
Other:
- board outline added: 40.2 x 26.2 mm

Commit message: finishedpcbdesign
Parts:
- added C1: 0.1μF, Capacitor_SMD:C_0805_2012Metric_Pad1.18x1.45mm_HandSolder, F.Cu at (128.1, 68.5)
Routing:
- net GND: track 14.0 -> 0.00 mm, vias 5 -> 6
Other:
- board text added: "0"
- board text added: "1"
- board text added: "2"
- board text added: "3"
- board text added: "3.3v"
- board text added: "4"
- board text added: "set"
