File: Switch Lock/Switch Lock.kicad_sch (KiCad schematic)
At the start: 6 parts, among them J1 Conn_01x06, SW1 SW_SPST, SW2 SW_SPST, SW3 SW_SPST, SW4 SW_SPST, SW5 SW_SPST

Commit message: 123
Parts:
- removed J1: Conn_01x06, Connector_PinHeader_2.54mm:PinHeader_1x06_P2.54mm_Vertical, symbol Connector_Generic:Conn_01x06
- removed SW1, SW2, SW3, SW4, SW5: SW_SPST, symbol Switch:SW_SPST
- added J2: Conn_01x07, symbol Connector_Generic:Conn_01x07
- added R1: 2.2k, Resistor_SMD:R_0805_2012Metric_Pad1.20x1.40mm_HandSolder, symbol Device:R_US
- added S1, S2, S3, S4, Status1: JS102011SAQN, JS102011SAQN:SW_JS102011SAQN, symbol SS_js102011:JS102011SAQN
Connections:
- new net: J2.1 (Pin_1), R1.2
- new net: J2.5 (Pin_5), S4.1
- new net: J2.2 (Pin_2), S1.1
- new net: J2.3 (Pin_3), S2.1
- new net: J2.4 (Pin_4), S3.1
- new net: J2.6 (Pin_6), Status1.1
- new net 3.3v: R1.1, S1.2, S2.2, S3.2, S4.2, Status1.2
- new net GND: J2.7 (Pin_7), S1.3, S2.3, S3.3, S4.3, Status1.3

Commit message: finisheddesign
Parts:
- J2: footprint (none) -> Connector_PinHeader_2.54mm:PinHeader_1x07_P2.54mm_Vertical
Changed lines of the file:
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@@
 			)
 		)
-		(property "Footprint" ""
+		(property "Footprint" "Connector_PinHeader_2.54mm:PinHeader_1x07_P2.54mm_Vertical"
 			(at 104.14 66.04 0)
 			(effects

Commit message: finishedpcbdesign
Parts:
- added C1: 0.1μF, Capacitor_SMD:C_0805_2012Metric_Pad1.18x1.45mm_HandSolder, symbol Device:C
Connections:
- net 3.3v: now also C1.2
- net GND: now also C1.1
Changed lines of the file:
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@@
+		)
+	)
+	(label "3.3v"
+		(at 113.03 88.9 0)
+		(fields_autoplaced yes)
+		(effects
+			(font
+				(size 1.27 1.27)
+			)
+			(justify left bottom)
 		)
 	)
@@
 		(property "Intersheetrefs" "${INTERSHEET_REFS}"
 			(at 56.6443 105.41 0)
+			(effects
+				(font
+					(size 1.27 1.27)
+				)
+				(justify right)
+				(hide yes)
+			)
+		)
+	)
+	(global_label "GND"
+		(shape input)
+		(at 105.41 88.9 180)
+		(fields_autoplaced yes)
+		(effects
+			(font
+				(size 1.27 1.27)
+			)
+			(justify right)
+		)
+		(property "Intersheetrefs" "${INTERSHEET_REFS}"
+			(at 98.5543 88.9 0)
 			(effects
 				(font
@@
 					(unit 1)
 				)
+			)
+		)
+	)
+	(symbol
+		(lib_id "Device:C")
+		(at 109.22 88.9 90)
+		(unit 1)
+		(exclude_from_sim no)
+		(in_bom yes)
+		(on_board yes)
+		(dnp no)
+		(fields_autoplaced yes)
+		(property "Reference" "C1"
+			(at 109.22 81.28 90)
+			(effects
+				(font
+					(size 1.27 1.27)
+				)
+			)
+		)
+		(property "Value" "0.1μF"
+			(at 109.22 83.82 90)
+			(effects
+				(font
+					(size 1.27 1.27)
+				)
+			)
+		)
+		(property "Footprint" "Capacitor_SMD:C_0805_2012Metric_Pad1.18x1.45mm_HandSolder"
+			(at 113.03 87.9348 0)
+			(effects
+				(font
+					(size 1.27 1.27)
+				)
+				(hide yes)
+			)
+		)
+		(property "Datasheet" "~"
+			(at 109.22 88.9 0)
+			(effects
+				(font
+					(size 1.27 1.27)
+				)
+				(hide yes)
+			)
+		)
+		(property "Description" "Unpolarized capacitor"
+			(at 109.22 88.9 0)
+			(effects
+				(font
+					(size 1.27 1.27)
+				)
+				(hide yes)
+			)
+		)
+		(pin "2"
+		)
+		(pin "1"
+		)
+		(instances
+			(project ""
+				(path "/a7de3e81-b9d9-4234-882c-494d456291b7"
+					(reference "C1")
+					(unit 1)
+				)

Commit message: 3dmodoling
Connections:
- net 3.3v: now also S1.1, S2.1, S3.1, S4.1, Status1.1; no longer S1.2, S2.2, S3.2, S4.2, Status1.2
- net at J2.5 (Pin_5): now also S4.2; no longer S4.1
- net at J2.2 (Pin_2): now also S1.2; no longer S1.1
- net at J2.3 (Pin_3): now also S2.2; no longer S2.1
- net at J2.4 (Pin_4): now also S3.2; no longer S3.1
- net at J2.6 (Pin_6): now also Status1.2; no longer Status1.1
Changed lines of the file:
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@@
 	(wire
 		(pts
-			(xy 63.5 49.53) (xy 53.34 49.53)
+			(xy 81.28 68.58) (xy 99.06 68.58)
 		)
 		(stroke
@@
 	(wire
 		(pts
-			(xy 78.74 67.31) (xy 78.74 64.77)
+			(xy 78.74 102.87) (xy 85.09 102.87)
 		)
 		(stroke
@@
 	(wire
 		(pts
-			(xy 63.5 62.23) (xy 63.5 63.5)
+			(xy 82.55 60.96) (xy 99.06 60.96)
 		)
 		(stroke
@@
 	(wire
 		(pts
-			(xy 53.34 49.53) (xy 53.34 60.96)
+			(xy 85.09 102.87) (xy 85.09 71.12)
 		)
 		(stroke
@@
 	(wire
 		(pts
-			(xy 86.36 66.04) (xy 99.06 66.04)
+			(xy 81.28 90.17) (xy 81.28 68.58)
 		)
 		(stroke
@@
 	(wire
 		(pts
-			(xy 63.5 83.82) (xy 87.63 83.82)
+			(xy 85.09 71.12) (xy 99.06 71.12)
 		)
 		(stroke
@@
 	(wire
 		(pts
-			(xy 81.28 67.31) (xy 78.74 67.31)
+			(xy 82.55 64.77) (xy 82.55 63.5)
 		)
 		(stroke
@@
 	(wire
 		(pts
-			(xy 88.9 96.52) (xy 88.9 71.12)
+			(xy 78.74 64.77) (xy 82.55 64.77)
 		)
 		(stroke
@@
 	(wire
 		(pts
-			(xy 86.36 58.42) (xy 91.44 58.42)
+			(xy 78.74 66.04) (xy 78.74 77.47)
 		)
 		(stroke
@@
 	(wire
 		(pts
-			(xy 53.34 60.96) (xy 99.06 60.96)
+			(xy 78.74 90.17) (xy 81.28 90.17)
 		)
 		(stroke
@@
 	(wire
 		(pts
-			(xy 63.5 96.52) (xy 88.9 96.52)
+			(xy 82.55 63.5) (xy 99.06 63.5)
 		)
 		(stroke
@@
 	(wire
 		(pts
-			(xy 87.63 68.58) (xy 99.06 68.58)
+			(xy 78.74 52.07) (xy 82.55 52.07)
 		)
 		(stroke
@@
 	(wire
 		(pts
-			(xy 63.5 71.12) (xy 86.36 71.12)
+			(xy 82.55 52.07) (xy 82.55 60.96)
 		)
 		(stroke
@@
 	(wire
 		(pts
-			(xy 63.5 74.93) (xy 63.5 71.12)
+			(xy 87.63 58.42) (xy 91.44 58.42)
 		)
 		(stroke
@@
 	(wire
 		(pts
-			(xy 63.5 87.63) (xy 63.5 83.82)
-		)
-		(stroke
-			(width 0)
-			(type default)
-		)
-	)
-	(wire
-		(pts
-			(xy 88.9 71.12) (xy 99.06 71.12)
-		)
-		(stroke
-			(width 0)
-			(type default)
-		)
-	)
-	(wire
-		(pts
-			(xy 63.5 63.5) (xy 99.06 63.5)
-		)
-		(stroke
-			(width 0)
-			(type default)
-		)
-	)
-	(wire
-		(pts
-			(xy 63.5 100.33) (xy 63.5 96.52)
-		)
-		(stroke
-			(width 0)
-			(type default)
-		)
-	)
-	(wire
-		(pts
-			(xy 87.63 83.82) (xy 87.63 68.58)
-		)
-		(stroke
-			(width 0)
-			(type default)
-		)
-	)
-	(wire
-		(pts
-			(xy 86.36 71.12) (xy 86.36 66.04)
+			(xy 78.74 66.04) (xy 99.06 66.04)
 		)
 		(stroke
@@
 	)
 	(label "3.3v"
-		(at 78.74 52.07 0)
+		(at 63.5 87.63 0)
 		(fields_autoplaced yes)
 		(effects
@@
 	)
 	(label "3.3v"
-		(at 86.36 58.42 0)
+		(at 63.5 74.93 0)
 		(fields_autoplaced yes)
 		(effects
@@
 	)
 	(label "3.3v"
-		(at 78.74 77.47 0)
+		(at 63.5 62.23 0)
 		(fields_autoplaced yes)
 		(effects
@@
 	)
 	(label "3.3v"
-		(at 78.74 90.17 0)
+		(at 87.63 58.42 0)
 		(fields_autoplaced yes)
 		(effects
@@
 	)
 	(label "3.3v"
-		(at 81.28 67.31 0)
+		(at 63.5 49.53 0)
 		(fields_autoplaced yes)
 		(effects
@@
 	)
 	(label "3.3v"
-		(at 78.74 102.87 0)
+		(at 63.5 100.33 0)
 		(fields_autoplaced yes)
 		(effects
